File: Proto264.kicad_pcb (KiCad board)
At the start: 2 copper layers, 99.8 x 99.9 mm, 5 parts, among them CN1 C16-Exp-Port, J1 PIN_HEADER, J2 PIN_HEADER_GND, J3 PIN_HEADER_VCC, J4 PROTO_AREA

Commit message: Correct label
Other:
- board text added: "C2HI"
